File: UART-Module.kicad_pcb (KiCad board)
At the start: 2 copper layers, 99.8 x 99.8 mm, 12 parts, among them J1 Conn_01x02_Male, J2 Conn_01x02_Male, J3 Conn_02x30_Odd_Even, J4 DE9_Receptacle_MountingHoles, Q1 1.8432, U1 74HC02, U2 74HC21, U4 R65C51

Commit message: complete traces
Parts:
- removed C3: 30pF, Capacitor_SMD:C_0805_2012Metric_Pad1.18x1.45mm_HandSolder
- C1: footprint Capacitor_SMD:C_0805_2012Metric -> Capacitor_SMD:C_0805_2012Metric_Pad1.18x1.45mm_HandSolder
- C2: value 1uF -> 30pF; footprint Capacitor_SMD:C_0805_2012Metric -> Capacitor_SMD:C_0805_2012Metric_Pad1.18x1.45mm_HandSolder
- moved C1 45.8 mm to (161.4, 90.4)
- moved C2 28.0 mm to (133.5, 90.5)
- moved U4 6.17 mm to (154.6, 98.0), turned to -45 degrees
- moved J4 2.69 mm to (149.4, 66.0)
- moved R1 0.14 mm to (133.5, 100.3)
Connections:
- C2 pad 1: +5V -> GND
- C2 pad 2: GND -> XTLI
Routing:
- net +5V: track 294.5 -> 438.1 mm, vias 3 -> 10
- net R/~{W}: track 0.00 -> 89.7 mm, vias 0 -> 3
- net ~{IRQ}: track 0.00 -> 86.1 mm, vias 0 -> 2
- net GND: track 351.9 -> 429.5 mm, vias 0 -> 4
- net A0: track 0.00 -> 68.5 mm, vias 0 -> 2
- net ~{RESET}: track 0.00 -> 67.8 mm, vias 0 -> 2
- net A1: track 0.00 -> 59.7 mm, vias 0 -> 2
- net E: track 0.00 -> 57.5 mm, vias 0 -> 2
- net MAPPED_MEM: track 0.00 -> 54.4 mm, vias 0 -> 2
- net D0: track 0.00 -> 52.5 mm, vias 0 -> 2
- net A3: track 0.00 -> 49.8 mm, vias 0 -> 4
- net A2: track 0.00 -> 48.8 mm, vias 0 -> 2
- net D2: track 0.00 -> 48.1 mm, vias 0 -> 2
- net D1: track 0.00 -> 47.1 mm, vias 0 -> 2
- net A7: track 0.00 -> 42.3 mm, vias 0 -> 2
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Other:
- board text added: "ACIA Adapter Prototype Board"
- board text removed: "UART Adapter Prototype Board"

Commit message: fix chip select
Connections:
- U2 pad 8: ~{CS1} -> CS0
- U4 pad 2: +5V -> CS0
- U4 pad 3: ~{CS1} -> GND
Routing:
- net ~{CS1}: track 24.0 -> 0.00 mm, vias 1 -> 0
- net CS0: track 0.00 -> 22.7 mm, vias 0 -> 1
- net +5V: track 438.1 -> 423.4 mm, vias 10 -> 7
- net A3: track 49.8 -> 47.0 mm, vias 4 -> 2
- net GND: track 429.5 -> 432.1 mm
- net A2: track 48.8 -> 46.3 mm, vias 2 -> 0
- net MAPPED_MEM: track 54.4 -> 52.3 mm
- added copper zone on B.Cu, net GND
- added copper zone on F.Cu, net GND
- removed copper zone on B.Cu, net (none)
- removed copper zone on F.Cu, net (none)

Commit message: add max232 for correct serial voltages
Parts:
- added C3: 0.1uF, Capacitor_THT:CP_Radial_Tantal_D4.5mm_P5.00mm, F.Cu at (157.2, 58.9)
- added C4: 0.1uF, Capacitor_THT:CP_Radial_Tantal_D4.5mm_P5.00mm, F.Cu at (152.9, 58.9)
- added C5: 0.1uF, Capacitor_THT:CP_Radial_Tantal_D4.5mm_P5.00mm, F.Cu at (137.0, 79.3)
- added C6: 0.1uF, Capacitor_THT:CP_Radial_Tantal_D4.5mm_P5.00mm, F.Cu at (136.7, 57.7)
- added C7: 0.1uF, Capacitor_THT:CP_Radial_Tantal_D4.5mm_P5.00mm, F.Cu at (136.7, 66.2)
- added U3: MAX232ID, Package_SO:SOIC-16W_7.5x10.3mm_P1.27mm, F.Cu at (149.8, 68.8)
- moved J4 22.2 mm to (171.5, 64.1), turned to 90 degrees
Connections:
- J4 pad 2: RxD -> RxDv
- J4 pad 3: TxD -> TxDv
Routing:
- net ~{RTS}: track 30.1 -> 62.0 mm, vias 1 -> 3
- net ~{CTS}: track 30.5 -> 61.8 mm, vias 1 -> 5
- net ~{DCD}: track 40.7 -> 65.6 mm, vias 0 -> 3
- net ~{DSR}: track 38.0 -> 62.4 mm, vias 2 -> 3
- net ~{DTR}: track 34.8 -> 58.8 mm, vias 1 -> 4
- net +5V: track 423.4 -> 443.6 mm
- net TxDv: track 0.00 -> 19.8 mm, vias 0 -> 3
- net RxDv: track 0.00 -> 18.5 mm, vias 0 -> 3
- net Net-(U3-C1+): track 0.00 -> 11.2 mm, vias 0 -> 1
- net Net-(U3-C1-): track 0.00 -> 10.1 mm, vias 0 -> 1
- net GND: track 432.1 -> 422.2 mm, vias 4 -> 9
- net Net-(U3-VS-): track 0.00 -> 9.58 mm, vias 0 -> 1
- net Net-(U3-C2+): track 0.00 -> 9.23 mm, vias 0 -> 1
- net Net-(U3-C2-): track 0.00 -> 9.12 mm, vias 0 -> 1
- net Net-(U3-VS+): track 0.00 -> 8.50 mm
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
Commit message: fix footprint for U3
Parts:
- U3: footprint Package_SO:SOIC-16W_7.5x10.3mm_P1.27mm -> Package_SO:SOIC-16_4.55x10.3mm_P1.27mm
Routing:
- net RxD: track 43.0 -> 41.3 mm
- net TxDv: track 19.8 -> 21.2 mm
- net TxD: track 38.9 -> 37.4 mm
- net GND: track 422.2 -> 423.6 mm
- net Net-(U3-VS-): track 9.58 -> 11.0 mm
- net Net-(U3-C2-): track 9.12 -> 10.5 mm
- net Net-(U3-C2+): track 9.23 -> 10.6 mm
- net Net-(U3-C1-): track 10.1 -> 11.5 mm
- net Net-(U3-C1+): track 11.2 -> 12.6 mm
- net RxDv: track 18.5 -> 19.9 mm
- net +5V: track 443.6 -> 443.1 mm
Other:
- board text added: "ACIA Adapter Board"
- board text added: "Rev 1.2"
- board text removed: "ACIA Adapter Prototype Board"
- board text removed: "Rev 1.1"
